File: pck100clone.brd (EAGLE design)
At the start: 72.4 x 68.6 mm, 90 parts, among them IC1 LM358N, IC3 LM358N, IC4 LM358N, IC5 LM358N, Q1 2SC945, Q2 2SC945, Q3 2N3906, Q4 2N3906, Q5 2N3904, Q6 2N3904

Commit message: rev2
Parts:
- moved OUT 1.42 mm to (17.8, 66.7), turned to 90 degrees
- moved 9VDC 1.42 mm to (72.4, 66.7), turned to 90 degrees
- moved R3 0.64 mm to (17.8, 62.2)
- moved R4 0.64 mm to (17.8, 59.7)
- moved C10 0.38 mm to (26.7, 55.5)
- moved C14 0.38 mm to (21.0, 55.5)
- moved C3 0.38 mm to (15.2, 55.5)
Connections:
- net GND: now also CLICK.3
Routing:
- net VCC: track 220.7 -> 219.3 mm
- net N$51: track 6.61 -> 5.99 mm
Changed lines of the file:
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@@
 <wire x1="8.89" y1="3.81" x2="8.89" y2="67.31" width="0.254" layer="20"/>
 <wire x1="8.89" y1="67.31" x2="11.43" y2="69.85" width="0.254" layer="20" curve="-90"/>
-<text x="15.367" y="65.405" size="1.27" layer="21" rot="R180">TIP</text>
+<text x="22.225" y="66.04" size="1.27" layer="21" rot="R180">TIP</text>
 <wire x1="15.24" y1="46.609" x2="38.735" y2="46.609" width="0.254" layer="21"/>
 <wire x1="38.735" y1="46.609" x2="38.735" y2="49.911" width="0.254" layer="21"/>
@@
 <text x="31.877" y="65.786" size="3.048" layer="21" font="vector">PCLONE-2</text>
 <text x="56.134" y="7.493" size="1.27" layer="21">LFO</text>
-<circle x="70.485" y="64.77" radius="1.135921875" width="0.4064" layer="21"/>
-<wire x1="69.85" y1="64.77" x2="71.12" y2="64.77" width="0.4064" layer="21"/>
-<wire x1="70.485" y1="65.405" x2="70.485" y2="64.135" width="0.4064" layer="21"/>
-<circle x="76.581" y="64.643" radius="1.135921875" width="0.4064" layer="21"/>
-<wire x1="75.946" y1="64.643" x2="77.216" y2="64.643" width="0.4064" layer="21"/>
+<circle x="69.215" y="65.405" radius="1.135921875" width="0.4064" layer="21"/>
+<wire x1="68.58" y1="65.405" x2="69.85" y2="65.405" width="0.4064" layer="21"/>
+<wire x1="69.215" y1="66.04" x2="69.215" y2="64.77" width="0.4064" layer="21"/>
+<circle x="69.215" y="67.945" radius="1.135921875" width="0.4064" layer="21"/>
+<wire x1="68.58" y1="67.945" x2="69.85" y2="67.945" width="0.4064" layer="21"/>
 <circle x="37.719" y="49.022" radius="0.359209375" width="0.4064" layer="21"/>
 <wire x1="20.955" y1="6.35" x2="20.955" y2="2.032" width="0.254" layer="21"/>
@@
 <attribute name="NAME" x="60.579" y="57.277" size="1.27" layer="25" ratio="10"/>
 </element>
-<element name="C14" library="rcl" package="E2,5-5" value="100/16" x="20.955" y="55.88" smashed="yes">
-<attribute name="NAME" x="16.383" y="52.197" size="1.27" layer="25" ratio="10"/>
+<element name="C14" library="rcl" package="E2,5-5" value="100/16" x="20.955" y="55.499" smashed="yes">
+<attribute name="NAME" x="18.796" y="50.673" size="1.27" layer="25" ratio="10" rot="R90"/>
 </element>
 <element name="R23" library="rcl" package="0207/7" value="47k" x="46.99" y="38.1" smashed="yes">
@@
 <attribute name="NAME" x="62.992" y="52.07" size="1.27" layer="25" ratio="10" rot="R180"/>
 </element>
-<element name="C10" library="rcl" package="E2,5-5" value="100/16" x="26.67" y="55.88" smashed="yes">
-<attribute name="NAME" x="23.749" y="58.547" size="1.27" layer="25" ratio="10"/>
+<element name="C10" library="rcl" package="E2,5-5" value="100/16" x="26.67" y="55.499" smashed="yes">
+<attribute name="NAME" x="25.273" y="58.293" size="1.27" layer="25" ratio="10"/>
 </element>
 <element name="D1" library="diode" package="DO41-10" value="1N4004" x="28.956" y="61.468" smashed="yes" rot="R180">
@@
 <attribute name="NAME" x="66.929" y="54.864" size="1.27" layer="25" ratio="10" rot="R180"/>
 </element>
-<element name="C3" library="rcl" package="E2,5-5" value="1/50" x="15.24" y="55.88" smashed="yes">
-<attribute name="NAME" x="11.176" y="52.324" size="1.27" layer="25" ratio="10"/>
-</element>
-<element name="R3" library="rcl" package="0207/7" value="10k" x="17.78" y="62.865" smashed="yes" rot="R180">
-<attribute name="NAME" x="17.78" y="63.373" size="1.27" layer="25" ratio="10" rot="R180"/>
-</element>
-<element name="R4" library="rcl" package="0207/7" value="47k" x="17.78" y="60.325" smashed="yes">
-<attribute name="NAME" x="15.875" y="59.817" size="1.27" layer="25" ratio="10"/>
+<element name="C3" library="rcl" package="E2,5-5" value="1/50" x="15.24" y="55.499" smashed="yes">
+<attribute name="NAME" x="13.208" y="51.562" size="1.27" layer="25" ratio="10" rot="R90"/>
+</element>
+<element name="R3" library="rcl" package="0207/7" value="10k" x="17.78" y="62.23" smashed="yes" rot="R180">
+<attribute name="NAME" x="17.78" y="62.738" size="1.27" layer="25" ratio="10" rot="R180"/>
+</element>
+<element name="R4" library="rcl" package="0207/7" value="47k" x="17.78" y="59.69" smashed="yes">
+<attribute name="NAME" x="15.875" y="59.182" size="1.27" layer="25" ratio="10"/>
 </element>
 <element name="PWR" library="led" package="LED3MM" value="" x="12.7" y="34.29" smashed="yes" rot="R270">
@@
 <attribute name="NAME" x="38.735" y="35.56" size="1.27" layer="25" ratio="10" rot="R270"/>
 </element>
-<element name="9VDC" library="pinhead" package="1X02" value="" x="73.66" y="67.31" smashed="yes">
-<attribute name="NAME" x="65.9638" y="66.7258" size="1.27" layer="25" ratio="10"/>
-<attribute name="VALUE" x="71.12" y="64.135" size="1.27" layer="27"/>
-</element>
-<element name="OUT" library="pinhead" package="1X02" value="" x="16.51" y="67.31" smashed="yes" rot="R180">
-<attribute name="NAME" x="23.1902" y="68.0212" size="1.27" layer="25" ratio="10" rot="R180"/>
-<attribute name="VALUE" x="19.05" y="70.485" size="1.27" layer="27" rot="R180"/>
+<element name="9VDC" library="pinhead" package="1X02" value="" x="72.39" y="66.675" smashed="yes" rot="R90">
+<attribute name="NAME" x="74.3458" y="69.2912" size="1.27" layer="25" ratio="10" rot="R270"/>
+<attribute name="VALUE" x="75.565" y="64.135" size="1.27" layer="27" rot="R90"/>
+</element>
+<element name="OUT" library="pinhead" package="1X02" value="" x="17.78" y="66.675" smashed="yes" rot="R90">
+<attribute name="NAME" x="15.9512" y="65.0748" size="1.27" layer="25" ratio="10" rot="R90"/>
+<attribute name="VALUE" x="20.955" y="64.135" size="1.27" layer="27" rot="R90"/>
 </element>
 <element name="SWEEP" library="pinhead" package="1X04" value="" x="48.895" y="3.81" smashed="yes">
@@
 <contactref element="9VDC" pad="2"/>
 <contactref element="OUT" pad="2"/>
+<contactref element="CLICK" pad="3"/>
 </signal>
 <signal name="N$1">
@@
 <wire x1="11.43" y1="46.99" x2="11.43" y2="35.56" width="0.4064" layer="1"/>
 <wire x1="15.24" y1="48.26" x2="15.24" y2="51.435" width="0.4064" layer="16"/>
-<wire x1="15.24" y1="51.435" x2="19.685" y2="55.88" width="0.4064" layer="16"/>
-<wire x1="19.685" y1="55.88" x2="19.685" y2="56.515" width="0.4064" layer="1"/>
+<wire x1="15.24" y1="51.435" x2="19.685" y2="55.499" width="0.4064" layer="16"/>
+<wire x1="19.685" y1="55.499" x2="19.685" y2="56.515" width="0.4064" layer="1"/>
 <wire x1="19.685" y1="56.515" x2="20.955" y2="57.785" width="0.4064" layer="1"/>
 <wire x1="20.955" y1="57.785" x2="25.4" y2="57.785" width="0.4064" layer="1"/>
@@
 <wire x1="24.13" y1="21.59" x2="22.86" y2="21.59" width="0.4064" layer="1"/>
 <wire x1="12.7" y1="35.56" x2="11.43" y2="35.56" width="0.4064" layer="1"/>
-<wire x1="25.4" y1="55.88" x2="25.4" y2="57.785" width="0.4064" layer="1"/>
+<wire x1="25.4" y1="55.499" x2="25.4" y2="57.785" width="0.4064" layer="1"/>
 <wire x1="27.94" y1="57.785" x2="32.385" y2="62.23" width="0.4064" layer="1"/>
 <wire x1="76.2" y1="55.88" x2="74.93" y2="55.88" width="0.4064" layer="1"/>
@@
 <wire x1="34.036" y1="61.976" x2="34.29" y2="62.23" width="0.4064" layer="1"/>
 <contactref element="9VDC" pad="1"/>
-<wire x1="72.39" y1="67.31" x2="72.39" y2="62.865" width="0.4064" layer="1"/>
 <wire x1="72.39" y1="62.865" x2="71.755" y2="62.23" width="0.4064" layer="1"/>
+<wire x1="72.39" y1="62.865" x2="72.39" y2="65.405" width="0.4064" layer="1"/>
 </signal>
 <signal name="N$10">
@@
 <wire x1="67.31" y1="46.99" x2="68.58" y2="46.99" width="0.4064" layer="1"/>
 <wire x1="27.94" y1="51.435" x2="30.48" y2="51.435" width="0.4064" layer="1"/>
-<wire x1="22.225" y1="55.88" x2="22.225" y2="54.61" width="0.4064" layer="1"/>
+<wire x1="22.225" y1="55.499" x2="22.225" y2="54.61" width="0.4064" layer="1"/>
 <wire x1="22.225" y1="54.61" x2="22.86" y2="53.975" width="0.4064" layer="1"/>
 <wire x1="68.58" y1="49.53" x2="71.12" y2="49.53" width="0.4064" layer="1"/>
@@
 <contactref element="C3" pad="+"/>
 <contactref element="IC6" pad="8"/>
-<wire x1="13.97" y1="55.88" x2="13.97" y2="54.61" width="0.4064" layer="1"/>
+<wire x1="13.97" y1="55.499" x2="13.97" y2="54.61" width="0.4064" layer="1"/>
 <wire x1="13.97" y1="54.61" x2="17.78" y2="50.8" width="0.4064" layer="1"/>
 <wire x1="17.78" y1="50.8" x2="17.78" y2="48.26" width="0.4064" layer="1"/>
@@
 <contactref element="C3" pad="-"/>
 <contactref element="R4" pad="1"/>
-<wire x1="16.51" y1="55.88" x2="16.51" y2="59.69" width="0.4064" layer="1"/>
-<wire x1="13.97" y1="60.325" x2="15.875" y2="60.325" width="0.4064" layer="1"/>
-<wire x1="15.875" y1="60.325" x2="16.51" y2="59.69" width="0.4064" layer="1"/>
+<wire x1="13.97" y1="59.69" x2="15.24" y2="59.69" width="0.4064" layer="1"/>
+<wire x1="15.24" y1="59.69" x2="16.51" y2="58.42" width="0.4064" layer="1"/>
+<wire x1="16.51" y1="58.42" x2="16.51" y2="55.499" width="0.4064" layer="1"/>
 </signal>
 <signal name="OUT">
 <contactref element="R4" pad="2"/>
 <contactref element="R3" pad="1"/>
-<wire x1="21.59" y1="62.865" x2="21.59" y2="60.325" width="0.4064" layer="1"/>
+<wire x1="21.59" y1="62.23" x2="21.59" y2="59.69" width="0.4064" layer="1"/>
 <contactref element="OUT" pad="1"/>
-<wire x1="17.78" y1="67.31" x2="17.78" y2="66.675" width="0.4064" layer="1"/>
-<wire x1="17.78" y1="66.675" x2="21.59" y2="62.865" width="0.4064" layer="1"/>
+<wire x1="21.59" y1="62.23" x2="21.59" y2="63.5" width="0.4064" layer="1"/>
+<wire x1="21.59" y1="63.5" x2="20.955" y2="64.135" width="0.4064" layer="1"/>
+<wire x1="20.955" y1="64.135" x2="20.32" y2="64.77" width="0.4064" layer="1"/>
+<wire x1="17.78" y1="65.405" x2="19.685" y2="65.405" width="0.4064" layer="1"/>
+<wire x1="19.685" y1="65.405" x2="20.32" y2="64.77" width="0.4064" layer="1"/>
 </signal>
 <signal name="N$38">

Commit message: rev3
Parts:
- added JP100, JP101, JP102, JP103, JP104, JP105, JP106, JP107, JP108, JP109, JP110, JP111, JP112, JP113, JP114, JP115, JP116, JP117, JP118, JP119, JP120, JP121, JP122, JP123, JP124, JP125, JP126, JP127, JP128, JP129, JP130, JP131, JP132, JP133, JP134, JP135, JP136, JP14, JP143, JP144, JP145, JP15, JP16, JP17, JP18, JP19, JP2, JP20, JP21, JP22, JP23, JP24, JP25, JP26, JP27, JP28, JP29, JP3, JP30, JP31, JP32, JP33, JP34, JP35, JP36, JP37, JP38, JP39, JP4, JP40, JP41, JP42, JP43, JP44, JP45, JP46, JP47, JP48, JP49, JP5, JP50, JP51, JP52, JP53, JP54, JP55, JP56, JP57, JP58, JP59, JP6, JP60, JP61, JP62, JP63, JP64, JP65, JP66, JP67, JP68, JP69, JP7, JP70, JP71, JP72, JP73, JP74, JP75, JP76, JP77, JP78, JP79, JP80, JP81, JP82, JP83, JP84, JP85, JP86, JP87, JP88, JP89, JP90, JP91, JP92, JP93, JP94, JP95, JP96, JP97, JP98, JP99: (no value), pinhead:1X01
- R45: value 10k -> 4k7
- moved 9VDC 8.28 mm to (80.6, 67.3), turned to 0 degrees
- moved OUT 5.12 mm to (22.9, 67.3), turned to 0 degrees
- moved C3 2.54 mm to (12.7, 55.5)
- moved C14 1.27 mm to (19.7, 55.5)
Connections:
- new net N$100: JP120.1, JP122.1, JP123.1
- new net N$101: JP124.1, JP125.1, JP126.1
- new net N$102: JP127.1, JP128.1, JP132.1
- new net N$103: JP129.1, JP130.1, JP131.1
- new net N$104: JP133.1, JP134.1, JP135.1
- new net N$18: JP4.1, JP5.1, JP6.1
- new net N$50: JP14.1, JP15.1, JP19.1
- new net N$52: JP16.1, JP17.1, JP18.1
- new net N$53: JP20.1, JP21.1, JP25.1
- new net N$54: JP22.1, JP23.1, JP24.1
- new net N$55: JP26.1, JP27.1, JP31.1
- new net N$56: JP28.1, JP29.1, JP30.1
- new net N$57: JP32.1, JP33.1, JP34.1
- new net N$58: JP35.1, JP36.1, JP37.1
- new net N$59: JP38.1, JP39.1, JP40.1
- new net N$60: JP41.1, JP42.1, JP43.1
- new net N$64: JP53.1, JP54.1, JP55.1
- new net N$65: JP56.1, JP57.1, JP61.1
- new net N$67: JP62.1, JP63.1, JP67.1
- new net N$68: JP64.1, JP65.1, JP66.1
- new net N$69: JP68.1, JP69.1, JP73.1
- new net N$70: JP70.1, JP71.1, JP72.1
- new net N$71: JP74.1, JP75.1, JP76.1
- new net N$72: JP77.1, JP78.1, JP79.1
- new net N$73: JP136.1, JP80.1, JP81.1
- new net N$89: JP105.1, JP98.1, JP99.1
- new net N$90: JP82.1, JP83.1, JP89.1
- new net N$91: JP85.1, JP86.1, JP87.1
- new net N$92: JP101.1, JP102.1, JP103.1
- new net N$93: JP106.1, JP107.1, JP113.1
- new net N$94: JP109.1, JP110.1, JP111.1
- new net N$95: JP114.1, JP115.1, JP121.1
- new net N$96: JP117.1, JP118.1, JP119.1
- new net N$97: JP84.1, JP88.1, JP92.1
- new net N$98: JP100.1, JP104.1, JP96.1
- new net N$99: JP108.1, JP112.1, JP116.1
- net GND: now also JP47.1, JP48.1, JP49.1, JP50.1, JP51.1, JP52.1, JP90.1, JP91.1, JP93.1, JP94.1, JP95.1, JP97.1
- net VCC: now also JP143.1, JP144.1, JP145.1, JP2.1, JP3.1, JP44.1, JP45.1, JP46.1, JP58.1, JP59.1, JP60.1, JP7.1
Routing:
- net VCC: track 219.3 -> 290.2 mm
- net N$99: track 0.00 -> 5.08 mm
- net N$98: track 0.00 -> 5.08 mm
- net N$97: track 0.00 -> 5.08 mm
- net N$96: track 0.00 -> 5.08 mm
- net N$95: track 0.00 -> 5.08 mm
- net N$94: track 0.00 -> 5.08 mm
- net N$93: track 0.00 -> 5.08 mm
- net N$92: track 0.00 -> 5.08 mm
- net N$91: track 0.00 -> 5.08 mm
- net N$90: track 0.00 -> 5.08 mm
- net N$89: track 0.00 -> 5.08 mm
- net N$73: track 0.00 -> 5.08 mm
- net N$72: track 0.00 -> 5.08 mm
- net N$71: track 0.00 -> 5.08 mm
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Other:
- board size 72.4 x 68.6 mm -> 85.7 x 68.6 mm
- board text added: "+"
- board text added: "-"
- board text added: "1"
- board text added: "2"
- board text added: "3"
- board text added: "4"
- board text added: "5"
- board text added: "6"
- board text added: "A"
- board text added: "B"
- board text added: "C"
- board text added: "D"
- board text added: "E"
- board text added: "F"
- board text added: "G"
- board text added: "H"
- board text added: "I"
- board text added: "J"
- board text added: "K"
- board text added: "L"
- board text added: "M"
- board text added: "N"
- board text added: "O"
- board text added: "P"
- board text added: "Q"
- board text added: "R"
- board text added: "rev 3"
- board text removed: "rev 2"
