File: pck100clone.sch (EAGLE design)
At the start: 85 parts, among them IC1 LM358N, IC3 LM358N, IC4 LM358N, IC5 LM358N, Q1 2SC945, Q2 2SC945

Commit message: fixes
Parts:
- removed JP1: (no value), pinhead:PINHD-1X9
Connections:
- removed net N$44: JP1.1, R19.2
- removed net N$46: C11.-, JP1.2, R7.1
- removed net N$48: D3.A, JP1.5
- removed net N$49: C4.2, JP1.6, JP1.7, R8.1
- removed net N$52: C3.+, JP1.8
- new net BA662_1: R19.2
- new net BA662_2: C11.-, R7.1
- new net BA662_5: D3.A
- new net BA662_6_7: C4.2, R8.1
- new net BA662_8: C3.+
- net GND: now also IC4P.V-
- net N$19: now also IC5A.-IN; no longer IC5B.+IN
- net N$20: now also IC5A.OUT; no longer IC5B.OUT
- net N$23: now also IC5A.+IN; no longer IC5B.-IN
- net N$38: now also IC5B.-IN; no longer IC5A.-IN
- net N$40: now also IC5B.OUT; no longer IC5A.OUT
- net N$42: now also IC5B.+IN; no longer IC5A.+IN
- net VCC: now also IC4P.V+; no longer JP1.9
- net VCO_OUT: no longer JP1.3
- net VGND: no longer JP1.4
Other:
- moved on the sheet: C11, C3, C4, D3, IC5A, IC5B, R19, R25, R3, R4, R5, R6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

Commit message: more changes
Parts:
- added IC6: (no value), pinhead:PINHD-1X9
- added LED1: (no value), led:LED3MM
- added Q3, Q4: 2N3906, transistor-pnp:2N3906
- added Q5, Q6: 2N3904, transistor:2N3904
- added R100: 4k7, rcl:R-EU_0207/7
Connections:
- new net N$44: LED1.C, R100.2
- new net N$45: IC6.4, Q4.C
- new net N$48: Q3.B, Q3.C, Q4.B, Q5.C
- net BA662_1: now also Q5.B, Q6.B, Q6.C
- net BA662_2: now also IC6.2
- net BA662_5: now also IC6.5
- net BA662_6_7: now also IC6.6, IC6.7
- net BA662_8: now also IC6.8
- net GND: now also Q5.E, Q6.E, R100.1; no longer SWEEP.3
- net VCC: now also IC6.9, LED1.A, Q3.E, Q4.E
- net VCO_OUT: now also IC6.1
- net VGND: now also IC6.3, SWEEP.3

Commit message: stuff
Parts:
- renumbered LED1 to PWR
Changed lines of the file:
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@@
 <part name="GND27" library="supply1" deviceset="GND" device=""/>
 <part name="P+10" library="supply1" deviceset="VCC" device=""/>
-<part name="LED1" library="led" deviceset="LED" device="3MM"/>
+<part name="PWR" library="led" deviceset="LED" device="3MM"/>
 <part name="R100" library="rcl" deviceset="R-EU_" device="0207/7" value="4k7"/>
 <part name="P+11" library="supply1" deviceset="VCC" device=""/>
@@
 <instance part="GND27" gate="1" x="203.2" y="5.08"/>
 <instance part="P+10" gate="VCC" x="203.2" y="43.18"/>
-<instance part="LED1" gate="G$1" x="238.76" y="-76.2"/>
+<instance part="PWR" gate="G$1" x="238.76" y="-76.2"/>
 <instance part="R100" gate="G$1" x="238.76" y="-88.9" rot="R90"/>
 <instance part="P+11" gate="VCC" x="238.76" y="-68.58"/>
@@
 </segment>
 <segment>
-<pinref part="LED1" gate="G$1" pin="A"/>
+<pinref part="PWR" gate="G$1" pin="A"/>
 <pinref part="P+11" gate="VCC" pin="VCC"/>
 <wire x1="238.76" y1="-73.66" x2="238.76" y2="-71.12" width="0.1524" layer="91"/>
@@
 <segment>
 <pinref part="R100" gate="G$1" pin="2"/>
-<pinref part="LED1" gate="G$1" pin="C"/>
+<pinref part="PWR" gate="G$1" pin="C"/>
 <wire x1="238.76" y1="-83.82" x2="238.76" y2="-81.28" width="0.1524" layer="91"/>
 </segment>

Commit message: almost done?
Parts:
- added SENS: (no value), pot:TRIM_EU-CA6V
- renumbered ATTACK to ATTK, DECAY_POT to DECAY, EXT_INPUT to TRIG, EXT_POWER to DC_IN, MOD_DEPTH to MOD, MOD_RATE to RATE, MOD_WAVE_FORM to WAVE, SENS_POT to LEVEL, SWEEP_TYPE to DIR
Connections:
- net GND: now also SENS.A
- net N$2: now also SENS.E
- net N$3: now also SENS.S

Commit message: more fussing
Parts:
- removed LEVEL, VCO_WAVE: (no value), pinhead:PINHD-1X3
- added SENS_LEVEL: (no value), pot:TRIM_EU-CA6V
- added SHAPE: (no value), pinhead:PINHD-1X2
- SENS: device pot:TRIM_EU-CA6V -> pinhead:PINHD-1X3
- WAVE: device pinhead:PINHD-1X2 -> pinhead:PINHD-1X3
- renumbered ATTK to ATTACK
Connections:
- net GND: now also SENS.3, SENS_LEVEL.A; no longer LEVEL.3, SENS.A
- net MOD_OUT: now also SHAPE.2; no longer WAVE.2
- net N$15: now also SHAPE.1; no longer WAVE.1
- net N$2: now also SENS.1, SENS_LEVEL.E; no longer LEVEL.1, SENS.E
- net N$3: now also SENS.2, SENS_LEVEL.S; no longer LEVEL.2, SENS.S
- net N$39: now also WAVE.1; no longer VCO_WAVE.1
- net N$41: now also WAVE.3; no longer VCO_WAVE.3
- net N$43: now also WAVE.2; no longer VCO_WAVE.2
Changed lines of the file:
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@@
 <parts>
 <part name="TRIG" library="pinhead" deviceset="PINHD-1X3" device=""/>
-<part name="LEVEL" library="pinhead" deviceset="PINHD-1X3" device=""/>
+<part name="SENS" library="pinhead" deviceset="PINHD-1X3" device=""/>
 <part name="PIEZO" library="pinhead" deviceset="PINHD-1X2" device=""/>
 <part name="GND1" library="supply1" deviceset="GND" device=""/>
@@
 <part name="GND12" library="supply1" deviceset="GND" device=""/>
 <part name="GND13" library="supply1" deviceset="GND" device=""/>
-<part name="ATTK" library="pinhead" deviceset="PINHD-1X2" device=""/>
+<part name="ATTACK" library="pinhead" deviceset="PINHD-1X2" device=""/>
 <part name="IC5" library="linear" deviceset="LM358" device="N"/>
 <part name="C13" library="rcl" deviceset="C-EU" device="050-025X075" value=".022"/>
@@
 <part name="RATE" library="pinhead" deviceset="PINHD-1X3" device=""/>
 <part name="R37" library="rcl" deviceset="R-EU_" device="0207/7" value="330"/>
-<part name="WAVE" library="pinhead" deviceset="PINHD-1X2" device=""/>
+<part name="SHAPE" library="pinhead" deviceset="PINHD-1X2" device=""/>
 <part name="R41" library="rcl" deviceset="R-EU_" device="0207/7" value="47k"/>
 <part name="MOD" library="pinhead" deviceset="PINHD-1X3" device=""/>
@@
 <part name="R33" library="rcl" deviceset="R-EU_" device="0207/7" value="47k"/>
 <part name="R31" library="rcl" deviceset="R-EU_" device="0207/7" value="100k"/>
-<part name="VCO_WAVE" library="pinhead" deviceset="PINHD-1X3" device=""/>
+<part name="WAVE" library="pinhead" deviceset="PINHD-1X3" device=""/>
 <part name="R32" library="rcl" deviceset="R-EU_" device="0207/7" value="220k"/>
 <part name="R36" library="rcl" deviceset="R-EU_" device="0207/7" value="100k"/>
@@
 <part name="GND14" library="supply1" deviceset="GND" device=""/>
 <part name="P+12" library="supply1" deviceset="VCC" device=""/>
-<part name="SENS" library="pot" deviceset="TRIM_EU-" device="CA6V"/>
+<part name="SENS_LEVEL" library="pot" deviceset="TRIM_EU-" device="CA6V"/>
 </parts>
 <sheets>
@@
 <instances>
 <instance part="TRIG" gate="A" x="7.62" y="93.98" rot="R90"/>
-<instance part="LEVEL" gate="A" x="22.86" y="93.98" rot="R90"/>
+<instance part="SENS" gate="A" x="22.86" y="93.98" rot="R90"/>
 <instance part="PIEZO" gate="G$1" x="-5.08" y="93.98" rot="R90"/>
 <instance part="GND1" gate="1" x="-7.62" y="81.28"/>
@@
 <instance part="GND12" gate="1" x="220.98" y="78.74"/>
 <instance part="GND13" gate="1" x="205.74" y="78.74"/>
-<instance part="ATTK" gate="G$1" x="231.14" y="99.06" rot="R90"/>
+<instance part="ATTACK" gate="G$1" x="231.14" y="99.06" rot="R90"/>
 <instance part="IC5" gate="B" x="281.94" y="22.86" smashed="yes" rot="MR180">
 <attribute name="NAME" x="284.48" y="19.685" size="1.778" layer="95" rot="MR180"/>
@@
 </instance>
 <instance part="R37" gate="G$1" x="48.26" y="-38.1" rot="R270"/>
-<instance part="WAVE" gate="G$1" x="71.12" y="7.62"/>
+<instance part="SHAPE" gate="G$1" x="71.12" y="7.62"/>
 <instance part="R41" gate="G$1" x="55.88" y="-15.24" rot="R180"/>
 <instance part="MOD" gate="A" x="187.96" y="-15.24"/>
@@
 <instance part="R33" gate="G$1" x="248.92" y="-5.08" rot="R90"/>
 <instance part="R31" gate="G$1" x="266.7" y="35.56"/>
-<instance part="VCO_WAVE" gate="A" x="307.34" y="40.64" rot="R90"/>
+<instance part="WAVE" gate="A" x="307.34" y="40.64" rot="R90"/>
 <instance part="R32" gate="G$1" x="299.72" y="22.86"/>
 <instance part="R36" gate="G$1" x="269.24" y="12.7"/>
@@
 <instance part="GND14" gate="1" x="109.22" y="-167.64"/>
 <instance part="P+12" gate="VCC" x="109.22" y="-116.84"/>
-<instance part="SENS" gate="1" x="22.86" y="104.14" rot="MR270"/>
+<instance part="SENS_LEVEL" gate="1" x="22.86" y="104.14" rot="MR270"/>
 </instances>
 <busses>
@@
 <segment>
 <pinref part="GND3" gate="1" pin="GND"/>
-<pinref part="LEVEL" gate="A" pin="3"/>
+<pinref part="SENS" gate="A" pin="3"/>
 <wire x1="25.4" y1="83.82" x2="25.4" y2="91.44" width="0.1524" layer="91"/>
 <wire x1="25.4" y1="91.44" x2="25.4" y2="99.06" width="0.1524" layer="91"/>
@@
 <wire x1="25.4" y1="99.06" x2="30.48" y2="99.06" width="0.1524" layer="91"/>
 <wire x1="30.48" y1="99.06" x2="30.48" y2="104.14" width="0.1524" layer="91"/>
-<pinref part="SENS" gate="1" pin="A"/>
+<pinref part="SENS_LEVEL" gate="1" pin="A"/>
 <wire x1="30.48" y1="104.14" x2="27.94" y2="104.14" width="0.1524" layer="91"/>
 </segment>
@@
 <pinref part="TRIG" gate="A" pin="2"/>
 <wire x1="7.62" y1="91.44" x2="7.62" y2="86.36" width="0.1524" layer="91"/>
-<pinref part="LEVEL" gate="A" pin="1"/>
+<pinref part="SENS" gate="A" pin="1"/>
 <wire x1="7.62" y1="86.36" x2="20.32" y2="86.36" width="0.1524" layer="91"/>
 <wire x1="20.32" y1="86.36" x2="20.32" y2="91.44" width="0.1524" layer="91"/>
@@
 <wire x1="20.32" y1="99.06" x2="15.24" y2="99.06" width="0.1524" layer="91"/>
 <wire x1="15.24" y1="99.06" x2="15.24" y2="104.14" width="0.1524" layer="91"/>
-<pinref part="SENS" gate="1" pin="E"/>
+<pinref part="SENS_LEVEL" gate="1" pin="E"/>
 <wire x1="15.24" y1="104.14" x2="17.78" y2="104.14" width="0.1524" layer="91"/>
 </segment>
@@
 <net name="N$3" class="0">
 <segment>
-<pinref part="LEVEL" gate="A" pin="2"/>
+<pinref part="SENS" gate="A" pin="2"/>
 <wire x1="22.86" y1="91.44" x2="22.86" y2="86.36" width="0.1524" layer="91"/>
 <pinref part="C7" gate="G$1" pin="1"/>
 <wire x1="22.86" y1="86.36" x2="33.02" y2="86.36" width="0.1524" layer="91"/>
-<pinref part="SENS" gate="1" pin="S"/>
+<pinref part="SENS_LEVEL" gate="1" pin="S"/>
 <wire x1="22.86" y1="91.44" x2="22.86" y2="99.06" width="0.1524" layer="91"/>
 <junction x="22.86" y="91.44"/>
@@
 <wire x1="218.44" y1="93.98" x2="220.98" y2="93.98" width="0.1524" layer="91"/>
 <wire x1="220.98" y1="93.98" x2="220.98" y2="91.44" width="0.1524" layer="91"/>
-<pinref part="ATTK" gate="G$1" pin="1"/>
+<pinref part="ATTACK" gate="G$1" pin="1"/>
 <wire x1="220.98" y1="93.98" x2="228.6" y2="93.98" width="0.1524" layer="91"/>
 <wire x1="228.6" y1="93.98" x2="228.6" y2="96.52" width="0.1524" layer="91"/>
@@
 <net name="ATTACK_OUT" class="0">
 <segment>
-<pinref part="ATTK" gate="G$1" pin="2"/>
+<pinref part="ATTACK" gate="G$1" pin="2"/>
 <wire x1="231.14" y1="96.52" x2="231.14" y2="93.98" width="0.1524" layer="91"/>
 <wire x1="231.14" y1="93.98" x2="241.3" y2="93.98" width="0.1524" layer="91"/>
@@
 <wire x1="50.8" y1="10.16" x2="40.64" y2="10.16" width="0.1524" layer="91"/>
 <junction x="50.8" y="20.32"/>
-<pinref part="WAVE" gate="G$1" pin="1"/>
+<pinref part="SHAPE" gate="G$1" pin="1"/>
 <wire x1="50.8" y1="10.16" x2="68.58" y2="10.16" width="0.1524" layer="91"/>
 <junction x="50.8" y="10.16"/>
@@
 <pinref part="R41" gate="G$1" pin="1"/>
 <wire x1="60.96" y1="-15.24" x2="76.2" y2="-15.24" width="0.1524" layer="91"/>
-<pinref part="WAVE" gate="G$1" pin="2"/>
+<pinref part="SHAPE" gate="G$1" pin="2"/>
 <wire x1="68.58" y1="7.62" x2="60.96" y2="7.62" width="0.1524" layer="91"/>
 <wire x1="60.96" y1="7.62" x2="60.96" y2="-15.24" width="0.1524" layer="91"/>
@@
 <segment>
 <pinref part="R31" gate="G$1" pin="2"/>
-<pinref part="VCO_WAVE" gate="A" pin="1"/>
+<pinref part="WAVE" gate="A" pin="1"/>
 <wire x1="271.78" y1="35.56" x2="304.8" y2="35.56" width="0.1524" layer="91"/>
 <wire x1="304.8" y1="35.56" x2="304.8" y2="38.1" width="0.1524" layer="91"/>
@@
 <segment>
 <pinref part="R32" gate="G$1" pin="2"/>
-<pinref part="VCO_WAVE" gate="A" pin="3"/>
+<pinref part="WAVE" gate="A" pin="3"/>
 <wire x1="304.8" y1="22.86" x2="309.88" y2="22.86" width="0.1524" layer="91"/>
 <wire x1="309.88" y1="22.86" x2="309.88" y2="38.1" width="0.1524" layer="91"/>
@@
 <net name="N$43" class="0">
 <segment>
-<pinref part="VCO_WAVE" gate="A" pin="2"/>
+<pinref part="WAVE" gate="A" pin="2"/>
 <wire x1="307.34" y1="38.1" x2="307.34" y2="10.16" width="0.1524" layer="91"/>
 <pinref part="C12" gate="G$1" pin="+"/>

Commit message: tweaks
Parts:
- renumbered R100 to R44
Changed lines of the file:
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@@
 <part name="P+10" library="supply1" deviceset="VCC" device=""/>
 <part name="PWR" library="led" deviceset="LED" device="3MM"/>
-<part name="R100" library="rcl" deviceset="R-EU_" device="0207/7" value="4k7"/>
+<part name="R44" library="rcl" deviceset="R-EU_" device="0207/7" value="4k7"/>
 <part name="P+11" library="supply1" deviceset="VCC" device=""/>
 <part name="GND28" library="supply1" deviceset="GND" device=""/>
@@
 <instance part="P+10" gate="VCC" x="203.2" y="43.18"/>
 <instance part="PWR" gate="G$1" x="238.76" y="-76.2"/>
-<instance part="R100" gate="G$1" x="238.76" y="-88.9" rot="R90"/>
+<instance part="R44" gate="G$1" x="238.76" y="-88.9" rot="R90"/>
 <instance part="P+11" gate="VCC" x="238.76" y="-68.58"/>
 <instance part="GND28" gate="1" x="238.76" y="-99.06"/>
@@
 <segment>
 <pinref part="GND28" gate="1" pin="GND"/>
-<pinref part="R100" gate="G$1" pin="1"/>
+<pinref part="R44" gate="G$1" pin="1"/>
 <wire x1="238.76" y1="-96.52" x2="238.76" y2="-93.98" width="0.1524" layer="91"/>
 </segment>
@@
 <net name="N$44" class="0">
 <segment>
-<pinref part="R100" gate="G$1" pin="2"/>
+<pinref part="R44" gate="G$1" pin="2"/>
 <pinref part="PWR" gate="G$1" pin="C"/>
 <wire x1="238.76" y1="-83.82" x2="238.76" y2="-81.28" width="0.1524" layer="91"/>
