File: pclone-control.sch (EAGLE design)
At the start: 20 parts

Commit message: work in progress
Parts:
- added 9VDC, BATT, IN, OUT, PIEZO: (no value), pinhead:PINHD-1X2
- added INPUT, OUTPUT: TRUCONNECTJACK, jason_eagle6:TRUCONNECTJACK
- added LED1: (no value), led:LED3MM
- added ONOFF: (no value), pinhead:PINHD-1X3
- added R2: 4k7, rcl:R-EU_0207/7
- added U$4: 2.1MMJACKTHM, adafruit:2.1MMJACKTHM
Connections:
- new net N$15: BATT.1, ONOFF.2, U$4.TIP
- new net N$29: BATT.2, U$4.RING_SW
- new net N$30: 9VDC.1, ONOFF.3, R2.1
- new net N$31: LED1.A, R2.2
- new net N$32: OUT.2, OUTPUT.TIP
- new net N$33: INPUT.TIP_NC, PIEZO.2
- new net N$34: IN.2, INPUT.TIP
- net GND: now also 9VDC.2, IN.1, INPUT.RING, INPUT.RING_NC, INPUT.SLEEVE, LED1.C, OUT.1, OUTPUT.RING, OUTPUT.RING_NC, OUTPUT.SLEEVE, PIEZO.1, U$4.RING
Other:
- moved on the sheet: CLICK, DECAY, DIR, J1, J2, J3, J4, J5, J6, J7, J8, J9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
