File: pclone-control.brd (EAGLE design)
At the start: 72.4 x 68.6 mm, 20 parts

Commit message: stuff
Routing:
- net N$26: track 60.7 -> 64.2 mm
- net N$25: track 39.2 -> 41.7 mm
- net N$24: track 25.8 -> 24.9 mm
- net N$28: track 53.0 -> 52.3 mm
Changed lines of the file:
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@@
 <contactref element="PITCH" pad="A"/>
 <contactref element="J3" pad="1"/>
-<wire x1="11.43" y1="20.32" x2="15.24" y2="20.32" width="0.6096" layer="1"/>
-<wire x1="15.24" y1="20.32" x2="28.575" y2="6.985" width="0.6096" layer="1"/>
-<wire x1="28.575" y1="3.81" x2="28.575" y2="6.985" width="0.6096" layer="1"/>
+<wire x1="28.575" y1="3.81" x2="28.575" y2="5.334" width="0.6096" layer="1"/>
+<wire x1="11.43" y1="20.32" x2="13.589" y2="20.32" width="0.6096" layer="1"/>
+<wire x1="13.589" y1="20.32" x2="28.575" y2="5.334" width="0.6096" layer="1"/>
 </signal>
 <signal name="N$25">
 <contactref element="PITCH" pad="B"/>
 <contactref element="J3" pad="3"/>
-<wire x1="6.35" y1="20.32" x2="6.35" y2="22.86" width="0.6096" layer="1"/>
-<wire x1="6.35" y1="22.86" x2="7.62" y2="24.13" width="0.6096" layer="1"/>
-<wire x1="7.62" y1="24.13" x2="13.97" y2="24.13" width="0.6096" layer="1"/>
-<wire x1="13.97" y1="24.13" x2="33.655" y2="4.445" width="0.6096" layer="1"/>
-<wire x1="33.655" y1="3.81" x2="33.655" y2="4.445" width="0.6096" layer="1"/>
+<wire x1="33.655" y1="3.81" x2="33.655" y2="5.842" width="0.6096" layer="1"/>
+<wire x1="33.655" y1="5.842" x2="14.351" y2="25.146" width="0.6096" layer="1"/>
+<wire x1="14.351" y1="25.146" x2="7.112" y2="25.146" width="0.6096" layer="1"/>
+<wire x1="7.112" y1="25.146" x2="6.35" y2="24.384" width="0.6096" layer="1"/>
+<wire x1="6.35" y1="24.384" x2="6.35" y2="20.32" width="0.6096" layer="1"/>
 </signal>
 <signal name="N$27">
 <contactref element="LFO_RATE" pad="B"/>
 <contactref element="J7" pad="3"/>
-<wire x1="60.96" y1="45.72" x2="60.96" y2="46.99" width="0.6096" layer="1"/>
-<wire x1="60.96" y1="46.99" x2="63.5" y2="49.53" width="0.6096" layer="1"/>
-<wire x1="63.5" y1="49.53" x2="68.58" y2="49.53" width="0.6096" layer="1"/>
-<wire x1="68.58" y1="49.53" x2="69.85" y2="48.26" width="0.6096" layer="1"/>
-<wire x1="69.85" y1="48.26" x2="69.85" y2="44.45" width="0.6096" layer="1"/>
-<wire x1="69.85" y1="44.45" x2="64.389" y2="38.989" width="0.6096" layer="1"/>
-<wire x1="64.389" y1="38.989" x2="64.389" y2="28.575" width="0.6096" layer="1"/>
-<wire x1="64.389" y1="28.575" x2="64.516" y2="28.448" width="0.6096" layer="1"/>
-<wire x1="64.516" y1="28.448" x2="68.072" y2="28.448" width="0.6096" layer="1"/>
-<wire x1="68.072" y1="28.448" x2="70.358" y2="26.162" width="0.6096" layer="1"/>
-<wire x1="70.358" y1="26.162" x2="70.358" y2="18.288" width="0.6096" layer="1"/>
+<wire x1="70.358" y1="31.242" x2="70.358" y2="18.288" width="0.6096" layer="1"/>
 <wire x1="70.358" y1="18.288" x2="62.484" y2="10.414" width="0.6096" layer="1"/>
 <wire x1="62.484" y1="10.414" x2="62.484" y2="6.731" width="0.6096" layer="1"/>
 <wire x1="62.484" y1="6.731" x2="64.135" y2="5.08" width="0.6096" layer="1"/>
 <wire x1="64.135" y1="5.08" x2="64.135" y2="3.81" width="0.6096" layer="1"/>
+<wire x1="60.96" y1="45.72" x2="60.96" y2="49.53" width="0.6096" layer="1"/>
+<wire x1="60.96" y1="49.53" x2="62.23" y2="50.8" width="0.6096" layer="1"/>
+<wire x1="62.23" y1="50.8" x2="68.58" y2="50.8" width="0.6096" layer="1"/>
+<wire x1="70.358" y1="31.242" x2="66.04" y2="35.56" width="0.6096" layer="1"/>
+<wire x1="66.04" y1="35.56" x2="66.04" y2="39.37" width="0.6096" layer="1"/>
+<wire x1="66.04" y1="39.37" x2="69.85" y2="43.18" width="0.6096" layer="1"/>
+<wire x1="69.85" y1="43.18" x2="69.85" y2="49.53" width="0.6096" layer="1"/>
+<wire x1="69.85" y1="49.53" x2="68.58" y2="50.8" width="0.6096" layer="1"/>
 </signal>
 <signal name="N$28">
 <contactref element="LFO_RATE" pad="A"/>
 <contactref element="J7" pad="1"/>
-<wire x1="66.04" y1="45.72" x2="66.04" y2="43.18" width="0.6096" layer="1"/>
-<wire x1="66.04" y1="43.18" x2="64.77" y2="41.91" width="0.6096" layer="1"/>
-<wire x1="64.77" y1="41.91" x2="63.5" y2="41.91" width="0.6096" layer="1"/>
-<wire x1="63.5" y1="41.91" x2="62.23" y2="40.64" width="0.6096" layer="1"/>
 <wire x1="62.23" y1="40.64" x2="62.23" y2="27.94" width="0.6096" layer="1"/>
 <wire x1="62.23" y1="27.94" x2="63.5" y2="26.67" width="0.6096" layer="1"/>
@@
 <wire x1="60.706" y1="11.176" x2="60.706" y2="6.731" width="0.6096" layer="1"/>
 <wire x1="60.706" y1="6.731" x2="59.055" y2="5.08" width="0.6096" layer="1"/>
+<wire x1="66.04" y1="45.72" x2="66.04" y2="44.45" width="0.6096" layer="1"/>
+<wire x1="66.04" y1="44.45" x2="62.23" y2="40.64" width="0.6096" layer="1"/>
 </signal>
 <signal name="N$23">
 <contactref element="J3" pad="2"/>
 <contactref element="PITCH" pad="W"/>
-<wire x1="8.89" y1="20.32" x2="8.89" y2="21.59" width="0.6096" layer="1"/>
-<wire x1="8.89" y1="21.59" x2="10.16" y2="22.86" width="0.6096" layer="1"/>
-<wire x1="10.16" y1="22.86" x2="13.97" y2="22.86" width="0.6096" layer="1"/>
-<wire x1="13.97" y1="22.86" x2="31.115" y2="5.715" width="0.6096" layer="1"/>
 <wire x1="31.115" y1="3.81" x2="31.115" y2="5.715" width="0.6096" layer="1"/>
+<wire x1="31.115" y1="5.715" x2="13.97" y2="22.86" width="0.6096" layer="1"/>
+<wire x1="13.97" y1="22.86" x2="9.779" y2="22.86" width="0.6096" layer="1"/>
+<wire x1="9.779" y1="22.86" x2="8.89" y2="21.971" width="0.6096" layer="1"/>
+<wire x1="8.89" y1="21.971" x2="8.89" y2="20.32" width="0.6096" layer="1"/>
 </signal>
 <signal name="N$17">
@@
 <contactref element="J7" pad="2"/>
 <contactref element="LFO_RATE" pad="W"/>
-<wire x1="63.5" y1="45.72" x2="63.5" y2="46.99" width="0.6096" layer="1"/>
-<wire x1="63.5" y1="46.99" x2="64.77" y2="48.26" width="0.6096" layer="1"/>
-<wire x1="64.77" y1="48.26" x2="67.31" y2="48.26" width="0.6096" layer="1"/>
-<wire x1="67.31" y1="48.26" x2="68.58" y2="46.99" width="0.6096" layer="1"/>
-<wire x1="68.58" y1="46.99" x2="68.58" y2="44.45" width="0.6096" layer="1"/>
+<wire x1="68.58" y1="49.149" x2="68.58" y2="44.45" width="0.6096" layer="1"/>
 <wire x1="68.58" y1="44.45" x2="63.5" y2="39.37" width="0.6096" layer="1"/>
 <wire x1="63.5" y1="39.37" x2="63.5" y2="27.94" width="0.6096" layer="1"/>
@@
 <wire x1="69.469" y1="18.669" x2="61.595" y2="10.795" width="0.6096" layer="1"/>
 <wire x1="61.595" y1="3.81" x2="61.595" y2="10.795" width="0.6096" layer="1"/>
+<wire x1="63.5" y1="45.72" x2="63.5" y2="48.895" width="0.6096" layer="1"/>
+<wire x1="63.5" y1="48.895" x2="64.262" y2="49.657" width="0.6096" layer="1"/>
+<wire x1="64.262" y1="49.657" x2="68.072" y2="49.657" width="0.6096" layer="1"/>
+<wire x1="68.072" y1="49.657" x2="68.58" y2="49.149" width="0.6096" layer="1"/>
 </signal>
 <signal name="N$20">

Commit message: work in progress
Parts:
- added 9VDC, BATT, IN, OUT, PIEZO: (no value), pinhead:1X02
- added INPUT, OUTPUT: TRUCONNECTJACK, jason_eagle6:TRUCONNECTJACK
- added LED1: (no value), led:LED3MM
- added ONOFF: (no value), pinhead:1X03
- added R2: 4k7, rcl:0207/7
- added U$4: 2.1MMJACKTHM, adafruit:PJ-102A
- moved WAVE 25.5 mm to (54.6, 58.4)
- moved LFO_SHAPE 16.7 mm to (73.7, 58.4)
- moved DECAY 8.98 mm to (45.1, 36.8)
- moved J8 8.98 mm to (55.2, 43.2)
- moved J9 8.98 mm to (62.9, 43.2)
- moved LFO_RATE 8.98 mm to (72.4, 36.8)
- moved MOD 8.98 mm to (72.4, 14.0)
- moved PITCH 8.98 mm to (17.8, 14.0)
- moved R1 8.98 mm to (45.1, 25.7)
- moved SENS 8.98 mm to (17.8, 36.8)
- moved SWP 8.98 mm to (45.1, 14.0)
- moved J6 8.89 mm to (64.1, 3.81)
- moved J3 8.89 mm to (40.0, 3.81)
- moved J1 8.89 mm to (24.8, 3.81)
- moved J4 8.89 mm to (48.9, 3.81)
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Connections:
- new net N$15: BATT.1, ONOFF.2, U$4.TIP
- new net N$29: BATT.2, U$4.RING_SW
- new net N$30: 9VDC.1, ONOFF.3, R2.1
- new net N$31: LED1.A, R2.2
- new net N$32: OUT.2, OUTPUT.TIP
- new net N$33: INPUT.TIP_NC, PIEZO.2
- new net N$34: IN.2, INPUT.TIP
- net GND: now also 9VDC.2, IN.1, INPUT.RING, INPUT.RING_NC, INPUT.SLEEVE, LED1.K, OUT.1, OUTPUT.RING, OUTPUT.RING_NC, OUTPUT.SLEEVE, PIEZO.1, U$4.RING
Routing:
- net N$34: track 0.00 -> 71.9 mm, vias 0 -> 1
- net N$33: track 0.00 -> 56.2 mm
- net N$31: track 0.00 -> 44.8 mm
- net N$3: track 83.7 -> 55.1 mm, vias 1 -> 0
- net N$30: track 0.00 -> 28.2 mm
- net N$32: track 0.00 -> 27.7 mm
- net N$15: track 0.00 -> 23.9 mm
- net N$2: track 84.2 -> 61.8 mm, vias 1 -> 0
- net N$8: track 46.2 -> 24.8 mm
- net N$9: track 38.7 -> 20.1 mm
- net N$26: track 64.2 -> 46.7 mm
- net N$7: track 32.2 -> 15.5 mm
- net N$4: track 78.6 -> 65.9 mm
- net N$12: track 74.3 -> 62.4 mm
- net N$13: track 77.8 -> 66.4 mm
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Other:
- board size 72.4 x 68.6 mm -> 72.4 x 76.2 mm

Commit message: rev3forreal
Parts:
- moved PIEZO 6.51 mm to (17.8, 28.1), turned to 0 degrees
- moved R1 2.54 mm to (45.1, 28.2)
- moved CLICK 2.29 mm to (17.8, 56.5)
- moved LFO_SHAPE 2.29 mm to (72.4, 56.5)
- moved BATT 1.91 mm to (64.1, 61.0)
- moved DIR 1.91 mm to (35.6, 56.5)
- moved WAVE 1.91 mm to (54.6, 56.5)
- moved OUT 1.42 mm to (17.8, 66.7), turned to 90 degrees
- moved 9VDC 1.42 mm to (72.4, 66.7), turned to 90 degrees
- moved LED1 1.27 mm to (14.0, 73.7)
- moved MOD 1.27 mm to (72.4, 12.7)
- moved PITCH 1.27 mm to (17.8, 12.7)
- moved SWP 1.27 mm to (45.1, 12.7)
Routing:
- net N$33: track 56.2 -> 48.5 mm
- net N$30: track 28.2 -> 32.3 mm
- net N$11: track 46.9 -> 44.4 mm
- net N$1: track 23.4 -> 26.0 mm
- net N$10: track 50.8 -> 48.4 mm
- net N$13: track 66.4 -> 64.0 mm
- net N$3: track 55.1 -> 57.5 mm
- net N$12: track 62.4 -> 64.7 mm
- net N$2: track 61.8 -> 59.7 mm
- net N$31: track 44.8 -> 42.7 mm
- net N$15: track 23.9 -> 22.0 mm
- net N$5: track 75.0 -> 73.1 mm
- net N$9: track 20.1 -> 18.2 mm
- net N$8: track 24.8 -> 22.9 mm
- net N$7: track 15.5 -> 13.6 mm
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