File: panel/pclone2_panel.brd (EAGLE design)
At the start: 86 x 89 mm, 17 parts

Commit message: PANEL CHANGES
Parts:
- R1: value (none) -> 470
Other:
- board text added: "CLICK"
- board text added: "DECAY A1M"
- board text added: "DEPTH A100K"
- board text added: "GND"
- board text added: "LFO WAVE"
- board text added: "PCLONE2 CONTROL PANEL PCB V1"
- board text added: "PITCH A100K"
- board text added: "RATE A100K"
- board text added: "SENS A100K"
- board text added: "SIXTY FOUR PIXELS LTD"
- board text added: "SWEEP"
- board text added: "SWEEP B470R"
- board text added: "TRIG"
- board text added: "VCO WAVE"
