File: panel/pclone2_panel.brd (EAGLE design)
At the start: 86 x 89 mm, 17 parts

Commit message: asas
Parts:
- removed GND: (no value), jason_eagle6:PINHEADPAD
- removed JP2: (no value), microbuilder:1X05_SMT
- removed X2A: (no value), microbuilder:1X03_SMT
- removed X2B, X2C: (no value), microbuilder:1X10_SMT
- added ADECAY, CLK, MDEP, MRAT, TSENS, VPITCH, VSHP: (no value), pinhead:1X03
- added JP3: (no value), pinhead:1X20
- added JP4: (no value), pinhead:1X01
- added JP5: (no value), pinhead:1X06
- added MSHP, TIN: (no value), pinhead:1X02
- added VSWP: (no value), pinhead:1X04
- moved JP1 73.1 mm to (81.4, 12.6)
Connections:
- removed net DECAY1: X2B.8
- removed net TRIG1: X2A.3
- net CLICK1: now also CLK.2; no longer JP2.5
- net CLICK2: now also CLK.3; no longer JP2.4
- net DECAY2: now also ADECAY.2; no longer X2B.7
- net DECAY3: now also ADECAY.3; no longer X2B.6
- net DEPTH1: now also MDEP.1; no longer X2C.8
- net DEPTH2: now also MDEP.2; no longer X2C.7
- net DEPTH3: now also MDEP.3; no longer X2C.6
- net GND: now also ADECAY.1, CLK.1, TIN.1, TSENS.1; no longer GND.P$1
- net MODRATE1: now also MRAT.1; no longer X2C.3
- net MODRATE2: now also MRAT.2; no longer X2C.2
- net MODRATE3: now also MRAT.3; no longer X2C.1
- net MODSHAPE1: now also MSHP.1; no longer X2C.5
- net MODSHAPE2: now also MSHP.2; no longer X2C.4
- net PITCH1: now also VPITCH.1; no longer X2B.5
- net PITCH2: now also VPITCH.2; no longer X2B.4
- net PITCH3: now also VPITCH.3; no longer X2B.3
- net SENS1: no longer X2A.1
- net SENS2: now also TSENS.2; no longer X2B.10
- net SENS3: now also TSENS.3; no longer X2B.9
- net SWEEP1: now also VSWP.1; no longer X2B.2
- net SWEEP2: now also VSWP.2; no longer X2B.1
- net SWEEP3: now also VSWP.3; no longer X2C.10
- net SWEEP4: now also VSWP.4; no longer X2C.9
- net TRIG2: now also TIN.2; no longer X2A.2
- net VCOWAVE1: now also VSHP.1; no longer JP2.3
- net VCOWAVE2: now also VSHP.2; no longer JP2.2
- net VCOWAVE3: now also VSHP.3; no longer JP2.1
Routing:
- net SENS1: track 115.3 -> 0.00 mm, vias 3 -> 0
- net DEPTH1: track 108.9 -> 0.00 mm, vias 2 -> 0
- net SWEEP_B: track 107.4 -> 0.00 mm, vias 3 -> 0
- net MODSHAPE2: track 99.8 -> 0.00 mm, vias 2 -> 0
- net DECAY2: track 99.4 -> 0.00 mm, vias 2 -> 0
- net MODSHAPE1: track 99.3 -> 0.00 mm, vias 2 -> 0
- net SWEEP2: track 88.7 -> 0.00 mm, vias 2 -> 0
- net SWEEP4: track 87.0 -> 0.00 mm, vias 2 -> 0
- net PITCH3: track 80.7 -> 0.00 mm, vias 2 -> 0
- net CLICK1: track 78.5 -> 0.00 mm
- net VCOWAVE2: track 70.9 -> 0.00 mm
- net MODRATE1: track 69.5 -> 0.00 mm
- net VCOWAVE3: track 69.1 -> 0.00 mm, vias 2 -> 0
- net MODRATE2: track 66.9 -> 0.00 mm
- net CLICK2: track 63.2 -> 0.00 mm
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Other:
- board size 86 x 89 mm -> 86 x 88 mm

Commit message: dsfdfs
Parts:
- removed JP3: (no value), pinhead:1X20
- removed JP4: (no value), pinhead:1X01
- removed JP5: (no value), pinhead:1X06
- moved JP1 2.74 mm to (79.0, 14.0)
- moved R1 1.00 mm to (56.8, 73.3)
Connections:
- removed net DECAY2: ADECAY.2, DECAY.B, DECAY.W
- removed net DECAY3: ADECAY.3
- new net DECAY: ADECAY.2, ADECAY.3, DECAY.B, DECAY.W
Routing:
- net MODSHAPE1: track 0.00 -> 124.4 mm, vias 0 -> 2
- net MODSHAPE2: track 0.00 -> 121.5 mm, vias 0 -> 2
- net DEPTH1: track 0.00 -> 111.7 mm, vias 0 -> 2
- net SWEEP4: track 0.00 -> 98.4 mm, vias 0 -> 4
- net MODRATE3: track 0.00 -> 94.8 mm, vias 0 -> 1
- net SWEEP_B: track 0.00 -> 91.5 mm, vias 0 -> 3
- net SENS3: track 0.00 -> 90.7 mm, vias 0 -> 2
- net SENS2: track 0.00 -> 86.4 mm, vias 0 -> 2
- net PITCH3: track 0.00 -> 85.9 mm, vias 0 -> 3
- net SWEEP2: track 0.00 -> 85.5 mm, vias 0 -> 2
- net MODRATE2: track 0.00 -> 85.0 mm, vias 0 -> 1
- net MODRATE1: track 0.00 -> 79.8 mm, vias 0 -> 1
- net DECAY: track 0.00 -> 69.4 mm
- net SENS1: track 0.00 -> 63.7 mm, vias 0 -> 2
- net PITCH1: track 0.00 -> 61.3 mm, vias 0 -> 2
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Other:
- outline, holes or cut-outs redrawn
- board text removed: "GND"

Commit message: sdf
Parts:
- 470: value 470 -> (none)
- renumbered R1 to 470
Connections:
- net GND: no longer TSENS.1
- net MODSHAPE1: now also LFO_WAVE.B; no longer LFO_WAVE.A
- net SENS1: now also TSENS.1
- net VCOWAVE1: now also VCO_WAVE.B; no longer VCO_WAVE.A
- net VCOWAVE3: now also VCO_WAVE.A; no longer VCO_WAVE.B
Routing:
- net SENS1: track 63.7 -> 142.7 mm, vias 2 -> 5
- net VCOWAVE3: track 46.5 -> 33.8 mm
- net MODSHAPE1: track 124.4 -> 135.6 mm, vias 2 -> 4
- net VCOWAVE1: track 34.6 -> 44.0 mm
- net MODSHAPE2: track 121.5 -> 123.2 mm

Commit message: sad
Connections:
- removed net SENS1: DECAY.A, SENS.A, TSENS.1
- net GND: now also DECAY.A, SENS.A, TSENS.1
Routing:
- net SENS1: track 142.7 -> 0.00 mm, vias 5 -> 0
- net GND: track 0.00 -> 92.6 mm
Changed lines of the file:
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@@
 <vertex x="92" y="94"/>
 </polygon>
+<contactref element="DECAY" pad="A"/>
+<contactref element="SENS" pad="A"/>
+<contactref element="TSENS" pad="1"/>
+<wire x1="12.1" y1="45.9" x2="13" y2="45" width="0.4064" layer="16"/>
+<wire x1="13" y1="45" x2="15" y2="43" width="0.4064" layer="1"/>
+<wire x1="15" y1="43" x2="34" y2="43" width="0.4064" layer="1"/>
+<wire x1="51" y1="43" x2="62" y2="54" width="0.4064" layer="1"/>
+<wire x1="76.53" y1="7.15" x2="76.53" y2="9.47" width="0.4064" layer="16"/>
+<wire x1="76.53" y1="9.47" x2="75" y2="11" width="0.4064" layer="16"/>
+<wire x1="75" y1="11" x2="75" y2="17" width="0.4064" layer="16"/>
+<wire x1="75" y1="17" x2="74" y2="18" width="0.4064" layer="16"/>
+<wire x1="74" y1="18" x2="67" y2="18" width="0.4064" layer="16"/>
+<wire x1="67" y1="18" x2="64.5" y2="20.5" width="0.4064" layer="16"/>
+<wire x1="64.5" y1="20.5" x2="45.5" y2="20.5" width="0.4064" layer="1"/>
+<wire x1="45.5" y1="20.5" x2="43" y2="18" width="0.4064" layer="1"/>
+<wire x1="43" y1="18" x2="34" y2="18" width="0.4064" layer="1"/>
 </signal>
 <signal name="TRIG2">
@@
 <wire x1="79.07" y1="13.983" x2="79.032" y2="14.021" width="0.4064" layer="16"/>
 </signal>
-<signal name="SENS1">
-<contactref element="DECAY" pad="A"/>
-<contactref element="SENS" pad="A"/>
-<wire x1="12.1" y1="49.036" x2="12.1" y2="45.9" width="0.4064" layer="16"/>
-<wire x1="12.1" y1="45.9" x2="13" y2="45" width="0.4064" layer="16"/>
-<via x="13" y="45" extent="1-16" drill="0.6"/>
-<wire x1="13" y1="45" x2="15" y2="43" width="0.4064" layer="1"/>
-<wire x1="15" y1="43" x2="31" y2="43" width="0.4064" layer="1"/>
-<wire x1="34" y1="43" x2="51" y2="43" width="0.4064" layer="1"/>
-<wire x1="51" y1="43" x2="62" y2="54" width="0.4064" layer="1"/>
-<wire x1="62" y1="54" x2="62" y2="58" width="0.4064" layer="1"/>
-<via x="62" y="58" extent="1-16" drill="0.6"/>
-<wire x1="62" y1="58" x2="61.136" y2="58" width="0.4064" layer="16"/>
-<wire x1="61.136" y1="58" x2="61.1" y2="58.036" width="0.4064" layer="16"/>
-<contactref element="TSENS" pad="1"/>
-<wire x1="76.53" y1="7.15" x2="76.53" y2="9.47" width="0.4064" layer="16"/>
-<wire x1="76.53" y1="9.47" x2="75" y2="11" width="0.4064" layer="16"/>
-<wire x1="75" y1="11" x2="75" y2="17" width="0.4064" layer="16"/>
-<wire x1="75" y1="17" x2="74" y2="18" width="0.4064" layer="16"/>
-<wire x1="74" y1="18" x2="67" y2="18" width="0.4064" layer="16"/>
-<wire x1="67" y1="18" x2="64.5" y2="20.5" width="0.4064" layer="16"/>
-<via x="64.5" y="20.5" extent="1-16" drill="0.6"/>
-<wire x1="64.5" y1="20.5" x2="45.5" y2="20.5" width="0.4064" layer="1"/>
-<wire x1="45.5" y1="20.5" x2="43" y2="18" width="0.4064" layer="1"/>
-<wire x1="43" y1="18" x2="34" y2="18" width="0.4064" layer="1"/>
-<via x="34" y="18" extent="1-16" drill="0.6"/>
-<wire x1="34" y1="18" x2="34" y2="43" width="0.4064" layer="16"/>
-<via x="34" y="43" extent="1-16" drill="0.6"/>
-<wire x1="34" y1="43" x2="31" y2="43" width="0.4064" layer="1"/>
-</signal>
 <signal name="SENS2">

Commit message: 796
Connections:
- net SENS2: now also SENS.W; no longer SENS.B
- net SENS3: now also SENS.B; no longer SENS.W
- net SWEEP2: now also SWEEP_DIR.COM2; no longer SWEEP_DIR.COM1
- net SWEEP4: now also SWEEP_DIR.COM1; no longer SWEEP_DIR.COM2
Routing:
- net GND: track 92.6 -> 58.1 mm
- net SWEEP4: track 98.4 -> 112.1 mm, vias 4 -> 2
- net SENS2: track 86.4 -> 94.8 mm, vias 2 -> 4
- net SENS3: track 90.7 -> 85.1 mm
- net SWEEP2: track 85.5 -> 83.3 mm
- net N$1: track 40.9 -> 42.9 mm
- net DEPTH1: track 111.7 -> 111.1 mm

Commit message: sdsds
Parts:
- moved 470 1.00 mm to (56.8, 74.3)
Connections:
- removed net N$1: 470.2, SWEEP_DIR.A1, SWEEP_DIR.B2
- new net N$2: 470.2, SWEEP_DIR.A2, SWEEP_DIR.B1
- net SWEEP_B: now also SWEEP_DIR.A1, SWEEP_DIR.B2; no longer SWEEP_DIR.A2, SWEEP_DIR.B1
Routing:
- net N$1: track 42.9 -> 0.00 mm, vias 2 -> 0
- net N$2: track 0.00 -> 40.6 mm, vias 0 -> 3
- net SWEEP2: track 83.3 -> 90.7 mm
- net SWEEP_B: track 91.7 -> 94.4 mm
- net SWEEP4: track 112.1 -> 114.6 mm, vias 2 -> 4
- net DEPTH1: track 111.1 -> 113.1 mm
