File: panel/pclone2_panel.sch (EAGLE design)
At the start: 31 parts

Commit message: control panel board
Parts:
- removed 9VDC, BATT, IN, J6, OUT, PIEZO: (no value), pinhead:PINHD-1X2
- removed DIR: DPDT_SW, jason_eagle6:DPDT_SW
- removed INPUT, OUTPUT: TRUCONNECTJACK, jason_eagle6:TRUCONNECTJACK
- removed J1, J2, J3, J5, J7, J8, J9, ONOFF: (no value), pinhead:PINHD-1X3
- removed J4: (no value), pinhead:PINHD-1X4
- removed LED1: (no value), led:LED3MM
- removed LFO_RATE, MOD, SWP: ALPS_POT_SMALL, jasons_stuff:ALPS_POT_SMALL
- removed LFO_SHAPE, WAVE: SPDT_SW, jason_eagle6:SPDT_SW
- removed R2: 4k7, rcl:R-EU_0207/7
- removed U$4: 2.1MMJACKTHM, adafruit:2.1MMJACKTHM
- added DEPTH, RATE: A100K, jason_eagle6:16MM_POT_SMTD
- added GND, JP1: (no value), jason_eagle6:PINHD-1X1SMT
- added JP2: (no value), microbuilder:HEADER-1X5SMT
- added LFO_WAVE, VCO_WAVE: SPD_SMTD, jason_eagle6:SPD_SMTD
- added SWEEP: B470R, jason_eagle6:16MM_POT_SMTD
- added SWEEP_DIR: DPDT_SMTD, jason_eagle6:DPDT_SMTD
- added X2A: (no value), microbuilder:HEADER-1X3SMT
- added X2B, X2C: (no value), microbuilder:HEADER-1X10SMT
- CLICK: value SPDT_SW -> SPD_SMTD; device jason_eagle6:SPDT_SW -> jason_eagle6:SPD_SMTD
- DECAY: value ALPS_POT_SMALL -> A1M; device jasons_stuff:ALPS_POT_SMALL -> jason_eagle6:16MM_POT_SMTD
- PITCH, SENS: value ALPS_POT_SMALL -> A100K; device jasons_stuff:ALPS_POT_SMALL -> jason_eagle6:16MM_POT_SMTD
- R1: value 500R -> (none); device rcl:R-EU_0207/7 -> rcl:R-EU_R0805
Connections:
- removed net N$10: CLICK.B, J8.1
- removed net N$11: CLICK.COM, J8.2
- removed net N$12: J6.1, LFO_SHAPE.B
- removed net N$13: J6.2, LFO_SHAPE.COM
- removed net N$14: J1.2, SENS.W
- removed net N$15: BATT.1, ONOFF.2, U$4.TIP
- removed net N$16: J1.3, SENS.B
- removed net N$17: DECAY.W, J2.2
- removed net N$18: DECAY.A, J2.1
- removed net N$19: DECAY.B, J2.3
- removed net N$2: DIR.A1, DIR.B2, R1.1
- removed net N$20: J5.2, MOD.W
- removed net N$21: J5.1, MOD.A
- removed net N$22: J5.3, MOD.B
- removed net N$23: J3.2, PITCH.W
- removed net N$24: J3.1, PITCH.A
- removed net N$25: J3.3, PITCH.B
- removed net N$26: J7.2, LFO_RATE.W
- removed net N$27: J7.3, LFO_RATE.B
- removed net N$28: J7.1, LFO_RATE.A
- removed net N$29: BATT.2, U$4.RING_SW
- removed net N$3: DIR.A2, DIR.B1, SWP.A
- removed net N$30: 9VDC.1, ONOFF.3, R2.1
- removed net N$31: LED1.A, R2.2
- removed net N$32: OUT.2, OUTPUT.TIP
- removed net N$33: INPUT.TIP_NC, PIEZO.2
- removed net N$34: IN.2, INPUT.TIP
- removed net N$4: DIR.COM1, J4.4
- removed net N$5: DIR.COM2, J4.2
- removed net N$6: J4.3, SWP.W
- removed net N$7: J9.1, WAVE.B
- removed net N$8: J9.3, WAVE.A
- removed net N$9: J9.2, WAVE.COM
- new net CLICK1: CLICK.B, JP2.5
- new net CLICK2: CLICK.COM, JP2.4
- new net DECAY1: X2B.8
- new net DECAY2: DECAY.B, DECAY.W, X2B.7
- new net DECAY3: X2B.6
- new net DEPTH1: DEPTH.A, R1.1, SWEEP.A, X2C.8
- new net DEPTH2: DEPTH.W, X2C.7
- new net DEPTH3: X2C.6
- new net MODRATE1: RATE.A, X2C.3
- new net MODRATE2: RATE.W, X2C.2
- new net MODRATE3: RATE.B, X2C.1
- new net MODSHAPE1: LFO_WAVE.A, X2C.5
- new net MODSHAPE2: LFO_WAVE.COM, X2C.4
- new net PITCH1: PITCH.A, X2B.5
- new net PITCH2: PITCH.W, X2B.4
- new net PITCH3: DEPTH.B, PITCH.B, X2B.3
- new net SENS1: DECAY.A, SENS.A, X2A.1
- new net SENS2: SENS.B, X2B.10
- new net SENS3: SENS.W, X2B.9
- new net SWEEP1: X2B.2
- new net SWEEP2: SWEEP_DIR.COM1, X2B.1
- new net SWEEP3: SWEEP.W, X2C.10
- new net SWEEP4: SWEEP_DIR.COM2, X2C.9
- new net SWEEP_B: SWEEP.B, SWEEP_DIR.A2, SWEEP_DIR.B1
- new net TRIG1: X2A.3
- new net TRIG2: JP1.1, X2A.2
- new net VCOWAVE1: JP2.3, VCO_WAVE.A
- new net VCOWAVE2: JP2.2, VCO_WAVE.COM
- new net VCOWAVE3: JP2.1, VCO_WAVE.B
- net GND: now also CLICK.GND, DECAY.GND, DEPTH.GND, GND.1, LFO_WAVE.GND, PITCH.GND, RATE.GND, SENS.GND, SWEEP.GND, SWEEP_DIR.GND, VCO_WAVE.GND; no longer 9VDC.2, IN.1, INPUT.RING, INPUT.RING_NC, INPUT.SLEEVE, J1.1, LED1.C, OUT.1, OUTPUT.RING, OUTPUT.RING_NC, OUTPUT.SLEEVE, PIEZO.1, SENS.A, U$4.RING
- net N$1: now also SWEEP_DIR.A1, SWEEP_DIR.B2; no longer J4.1, SWP.B
Other:
- moved on the sheet: R1

Commit message: PANEL CHANGES
Parts:
- R1: value (none) -> 470
Changed lines of the file:
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@@
 <part name="GND10" library="supply1" deviceset="GND" device=""/>
 <part name="GND11" library="supply1" deviceset="GND" device=""/>
-<part name="R1" library="rcl" deviceset="R-EU_" device="R0805"/>
+<part name="R1" library="rcl" deviceset="R-EU_" device="R0805" value="470"/>
 <part name="JP1" library="jason_eagle6" deviceset="PINHD-1X1" device="SMT"/>
 <part name="GND" library="jason_eagle6" deviceset="PINHD-1X1" device="SMT"/>

Commit message: asas
Parts:
- removed GND: (no value), jason_eagle6:PINHD-1X1SMT
- removed JP2: (no value), microbuilder:HEADER-1X5SMT
- removed X2A: (no value), microbuilder:HEADER-1X3SMT
- removed X2B, X2C: (no value), microbuilder:HEADER-1X10SMT
- added ADECAY, CLK, MDEP, MRAT, TSENS, VPITCH, VSHP: (no value), pinhead:PINHD-1X3
- added JP3: (no value), pinhead:PINHD-1X20
- added JP4: (no value), pinhead:PINHD-1X1
- added JP5: (no value), pinhead:PINHD-1X6
- added MSHP, TIN: (no value), pinhead:PINHD-1X2
- added VSWP: (no value), pinhead:PINHD-1X4
Connections:
- removed net DECAY1: X2B.8
- removed net TRIG1: X2A.3
- net CLICK1: now also CLK.2; no longer JP2.5
- net CLICK2: now also CLK.3; no longer JP2.4
- net DECAY2: now also ADECAY.2; no longer X2B.7
- net DECAY3: now also ADECAY.3; no longer X2B.6
- net DEPTH1: now also MDEP.1; no longer X2C.8
- net DEPTH2: now also MDEP.2; no longer X2C.7
- net DEPTH3: now also MDEP.3; no longer X2C.6
- net GND: now also ADECAY.1, CLK.1, TIN.1, TSENS.1; no longer GND.1
- net MODRATE1: now also MRAT.1; no longer X2C.3
- net MODRATE2: now also MRAT.2; no longer X2C.2
- net MODRATE3: now also MRAT.3; no longer X2C.1
- net MODSHAPE1: now also MSHP.1; no longer X2C.5
- net MODSHAPE2: now also MSHP.2; no longer X2C.4
- net PITCH1: now also VPITCH.1; no longer X2B.5
- net PITCH2: now also VPITCH.2; no longer X2B.4
- net PITCH3: now also VPITCH.3; no longer X2B.3
- net SENS1: no longer X2A.1
- net SENS2: now also TSENS.2; no longer X2B.10
- net SENS3: now also TSENS.3; no longer X2B.9
- net SWEEP1: now also VSWP.1; no longer X2B.2
- net SWEEP2: now also VSWP.2; no longer X2B.1
- net SWEEP3: now also VSWP.3; no longer X2C.10
- net SWEEP4: now also VSWP.4; no longer X2C.9
- net TRIG2: now also TIN.2; no longer X2A.2
- net VCOWAVE1: now also VSHP.1; no longer JP2.3
- net VCOWAVE2: now also VSHP.2; no longer JP2.2
- net VCOWAVE3: now also VSHP.3; no longer JP2.1

Commit message: dsfdfs
Parts:
- removed JP3: (no value), pinhead:PINHD-1X20
- removed JP4: (no value), pinhead:PINHD-1X1
- removed JP5: (no value), pinhead:PINHD-1X6
Connections:
- removed net DECAY2: ADECAY.2, DECAY.B, DECAY.W
- removed net DECAY3: ADECAY.3
- new net DECAY: ADECAY.2, ADECAY.3, DECAY.B, DECAY.W
Changed lines of the file:
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@@
 <part name="R1" library="rcl" deviceset="R-EU_" device="R0805" value="470"/>
 <part name="JP1" library="jason_eagle6" deviceset="PINHD-1X1" device="SMT"/>
-<part name="JP3" library="pinhead" deviceset="PINHD-1X20" device=""/>
-<part name="JP4" library="pinhead" deviceset="PINHD-1X1" device=""/>
-<part name="JP5" library="pinhead" deviceset="PINHD-1X6" device=""/>
 <part name="MRAT" library="pinhead" deviceset="PINHD-1X3" device=""/>
 <part name="MSHP" library="pinhead" deviceset="PINHD-1X2" device=""/>
@@
 <instance part="R1" gate="G$1" x="86.36" y="116.84" rot="R90"/>
 <instance part="JP1" gate="G$1" x="121.92" y="-27.94"/>
-<instance part="JP3" gate="A" x="172.72" y="-30.48"/>
-<instance part="JP4" gate="G$1" x="213.36" y="-45.72"/>
-<instance part="JP5" gate="A" x="233.68" y="-30.48"/>
 <instance part="MRAT" gate="A" x="76.2" y="-68.58" smashed="yes">
 <attribute name="NAME" x="80.645" y="-72.39" size="1.778" layer="95" rot="R90"/>
@@
 </segment>
 </net>
-<net name="DECAY2" class="0">
+<net name="DECAY" class="0">
 <segment>
 <label x="55.88" y="-17.78" size="1.778" layer="95"/>
 <pinref part="ADECAY" gate="A" pin="2"/>
-<wire x1="58.42" y1="-17.78" x2="73.66" y2="-17.78" width="0.1524" layer="91"/>
+<wire x1="58.42" y1="-17.78" x2="68.58" y2="-17.78" width="0.1524" layer="91"/>
+<pinref part="ADECAY" gate="A" pin="3"/>
+<wire x1="68.58" y1="-17.78" x2="73.66" y2="-17.78" width="0.1524" layer="91"/>
+<wire x1="68.58" y1="-20.32" x2="73.66" y2="-20.32" width="0.1524" layer="91"/>
+<wire x1="68.58" y1="-17.78" x2="68.58" y2="-20.32" width="0.1524" layer="91"/>
+<junction x="68.58" y="-17.78"/>
 </segment>
 <segment>
@@
 </segment>
 </net>
-<net name="DECAY3" class="0">
-<segment>
-<label x="55.88" y="-20.32" size="1.778" layer="95"/>
-<pinref part="ADECAY" gate="A" pin="3"/>
-<wire x1="58.42" y1="-20.32" x2="73.66" y2="-20.32" width="0.1524" layer="91"/>
-</segment>
-</net>

Commit message: sdf
Parts:
- 470: value 470 -> (none)
- renumbered R1 to 470
Connections:
- net GND: no longer TSENS.1
- net MODSHAPE1: now also LFO_WAVE.B; no longer LFO_WAVE.A
- net SENS1: now also TSENS.1
- net VCOWAVE1: now also VCO_WAVE.B; no longer VCO_WAVE.A
- net VCOWAVE3: now also VCO_WAVE.A; no longer VCO_WAVE.B
Changed lines of the file:
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@@
 <part name="GND10" library="supply1" deviceset="GND" device=""/>
 <part name="GND11" library="supply1" deviceset="GND" device=""/>
-<part name="R1" library="rcl" deviceset="R-EU_" device="R0805" value="470"/>
+<part name="470" library="rcl" deviceset="R-EU_" device="R0805"/>
 <part name="JP1" library="jason_eagle6" deviceset="PINHD-1X1" device="SMT"/>
 <part name="MRAT" library="pinhead" deviceset="PINHD-1X3" device=""/>
@@
 <instance part="GND10" gate="1" x="111.76" y="121.92"/>
 <instance part="GND11" gate="1" x="111.76" y="88.9"/>
-<instance part="R1" gate="G$1" x="86.36" y="116.84" rot="R90"/>
+<instance part="470" gate="G$1" x="86.36" y="116.84" rot="R90"/>
 <instance part="JP1" gate="G$1" x="121.92" y="-27.94"/>
 <instance part="MRAT" gate="A" x="76.2" y="-68.58" smashed="yes">
@@
 <wire x1="58.42" y1="48.26" x2="58.42" y2="43.18" width="0.1524" layer="91"/>
 <label x="58.42" y="40.64" size="1.778" layer="95"/>
+</segment>
+<segment>
+<pinref part="TSENS" gate="A" pin="1"/>
+<wire x1="73.66" y1="-5.08" x2="58.42" y2="-5.08" width="0.1524" layer="91"/>
+<label x="55.88" y="-5.08" size="1.778" layer="95"/>
 </segment>
 </net>
@@
 </segment>
 <segment>
-<pinref part="R1" gate="G$1" pin="1"/>
+<pinref part="470" gate="G$1" pin="1"/>
 <wire x1="86.36" y1="111.76" x2="86.36" y2="109.22" width="0.1524" layer="91"/>
 <label x="83.82" y="106.68" size="1.778" layer="95"/>
@@
 </segment>
 <segment>
-<pinref part="LFO_WAVE" gate="G$1" pin="A"/>
-<wire x1="93.98" y1="99.06" x2="88.9" y2="99.06" width="0.1524" layer="91"/>
-<label x="78.74" y="99.06" size="1.778" layer="95"/>
+<label x="76.2" y="91.44" size="1.778" layer="95"/>
+<pinref part="LFO_WAVE" gate="G$1" pin="B"/>
+<wire x1="88.9" y1="93.98" x2="93.98" y2="93.98" width="0.1524" layer="91"/>
 </segment>
 </net>
@@
 <label x="55.88" y="2.54" size="1.778" layer="95"/>
 <pinref part="TIN" gate="G$1" pin="1"/>
-<wire x1="45.72" y1="-15.24" x2="45.72" y2="-5.08" width="0.1524" layer="91"/>
-<wire x1="45.72" y1="-5.08" x2="45.72" y2="2.54" width="0.1524" layer="91"/>
+<wire x1="45.72" y1="-15.24" x2="45.72" y2="2.54" width="0.1524" layer="91"/>
 <wire x1="45.72" y1="2.54" x2="73.66" y2="2.54" width="0.1524" layer="91"/>
-<label x="55.88" y="-5.08" size="1.778" layer="95"/>
-<pinref part="TSENS" gate="A" pin="1"/>
-<wire x1="45.72" y1="-5.08" x2="73.66" y2="-5.08" width="0.1524" layer="91"/>
-<junction x="45.72" y="-5.08"/>
 <label x="55.88" y="-15.24" size="1.778" layer="95"/>
 <pinref part="ADECAY" gate="A" pin="1"/>
@@
 </segment>
 <segment>
-<pinref part="VCO_WAVE" gate="G$1" pin="A"/>
-<wire x1="17.78" y1="134.62" x2="10.16" y2="134.62" width="0.1524" layer="91"/>
-<label x="2.54" y="134.62" size="1.778" layer="95"/>
+<label x="2.54" y="124.46" size="1.778" layer="95"/>
+<wire x1="17.78" y1="129.54" x2="10.16" y2="129.54" width="0.1524" layer="91"/>
+<pinref part="VCO_WAVE" gate="G$1" pin="B"/>
 </segment>
 </net>
@@
 </segment>
 <segment>
-<pinref part="VCO_WAVE" gate="G$1" pin="B"/>
-<wire x1="17.78" y1="129.54" x2="10.16" y2="129.54" width="0.1524" layer="91"/>
-<label x="2.54" y="129.54" size="1.778" layer="95"/>
+<label x="2.54" y="137.16" size="1.778" layer="95"/>
+<wire x1="17.78" y1="134.62" x2="10.16" y2="134.62" width="0.1524" layer="91"/>
+<pinref part="VCO_WAVE" gate="G$1" pin="A"/>
 </segment>
 </net>
@@
 <pinref part="SWEEP_DIR" gate="G$1" pin="A1"/>
 <wire x1="86.36" y1="142.24" x2="93.98" y2="142.24" width="0.1524" layer="91"/>
-<pinref part="R1" gate="G$1" pin="2"/>
+<pinref part="470" gate="G$1" pin="2"/>
 <wire x1="86.36" y1="121.92" x2="86.36" y2="127" width="0.1524" layer="91"/>
 <junction x="86.36" y="127"/>

Commit message: sad
Connections:
- removed net SENS1: DECAY.A, SENS.A, TSENS.1
- net GND: now also DECAY.A, SENS.A, TSENS.1
Changed lines of the file:
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@@
 <part name="GND12" library="supply1" deviceset="GND" device=""/>
 <part name="GND13" library="supply1" deviceset="GND" device=""/>
+<part name="GND1" library="supply1" deviceset="GND" device=""/>
+<part name="GND14" library="supply1" deviceset="GND" device=""/>
 </parts>
 <sheets>
@@
 <instance part="GND12" gate="1" x="104.14" y="-17.78"/>
 <instance part="GND13" gate="1" x="45.72" y="-81.28"/>
+<instance part="GND1" gate="1" x="83.82" y="40.64"/>
+<instance part="GND14" gate="1" x="58.42" y="40.64"/>
 </instances>
 <busses>
@@
 <pinref part="JP1" gate="G$1" pin="1"/>
 <wire x1="119.38" y1="-27.94" x2="88.9" y2="-27.94" width="0.1524" layer="91"/>
-</segment>
-</net>
-<net name="SENS1" class="0">
-<segment>
-<pinref part="DECAY" gate="G$1" pin="A"/>
-<wire x1="83.82" y1="48.26" x2="83.82" y2="43.18" width="0.1524" layer="91"/>
-<label x="83.82" y="40.64" size="1.778" layer="95"/>
-</segment>
-<segment>
-<pinref part="SENS" gate="G$1" pin="A"/>
-<wire x1="58.42" y1="48.26" x2="58.42" y2="43.18" width="0.1524" layer="91"/>
-<label x="58.42" y="40.64" size="1.778" layer="95"/>
-</segment>
-<segment>
-<pinref part="TSENS" gate="A" pin="1"/>
-<wire x1="73.66" y1="-5.08" x2="58.42" y2="-5.08" width="0.1524" layer="91"/>
-<label x="55.88" y="-5.08" size="1.778" layer="95"/>
 </segment>
 </net>
@@
 <label x="55.88" y="2.54" size="1.778" layer="95"/>
 <pinref part="TIN" gate="G$1" pin="1"/>
-<wire x1="45.72" y1="-15.24" x2="45.72" y2="2.54" width="0.1524" layer="91"/>
+<wire x1="45.72" y1="-15.24" x2="45.72" y2="-5.08" width="0.1524" layer="91"/>
+<wire x1="45.72" y1="-5.08" x2="45.72" y2="2.54" width="0.1524" layer="91"/>
 <wire x1="45.72" y1="2.54" x2="73.66" y2="2.54" width="0.1524" layer="91"/>
 <label x="55.88" y="-15.24" size="1.778" layer="95"/>
@@
 <wire x1="45.72" y1="-15.24" x2="73.66" y2="-15.24" width="0.1524" layer="91"/>
 <junction x="45.72" y="-15.24"/>
-</segment>
-</net>
+<pinref part="TSENS" gate="A" pin="1"/>
+<wire x1="73.66" y1="-5.08" x2="45.72" y2="-5.08" width="0.1524" layer="91"/>
+<label x="55.88" y="-5.08" size="1.778" layer="95"/>
+<junction x="45.72" y="-5.08"/>
+</segment>
+<segment>
+<pinref part="DECAY" gate="G$1" pin="A"/>
+<wire x1="83.82" y1="48.26" x2="83.82" y2="43.18" width="0.1524" layer="91"/>
+<pinref part="GND1" gate="1" pin="GND"/>
+</segment>
+<segment>
+<pinref part="SENS" gate="G$1" pin="A"/>
+<wire x1="58.42" y1="48.26" x2="58.42" y2="43.18" width="0.1524" layer="91"/>
+<pinref part="GND14" gate="1" pin="GND"/>
+</segment>
+</net>

Commit message: 796
Connections:
- net SENS2: now also SENS.W; no longer SENS.B
- net SENS3: now also SENS.B; no longer SENS.W
- net SWEEP2: now also SWEEP_DIR.COM2; no longer SWEEP_DIR.COM1
- net SWEEP4: now also SWEEP_DIR.COM1; no longer SWEEP_DIR.COM2
Changed lines of the file:
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@@
 </segment>
 <segment>
-<pinref part="SENS" gate="G$1" pin="B"/>
-<wire x1="58.42" y1="63.5" x2="58.42" y2="66.04" width="0.1524" layer="91"/>
-<label x="58.42" y="66.04" size="1.778" layer="95"/>
+<label x="66.04" y="53.34" size="1.778" layer="95"/>
+<pinref part="SENS" gate="G$1" pin="W"/>
+<wire x1="63.5" y1="55.88" x2="68.58" y2="55.88" width="0.1524" layer="91"/>
 </segment>
 </net>
@@
 </segment>
 <segment>
-<pinref part="SENS" gate="G$1" pin="W"/>
-<wire x1="63.5" y1="55.88" x2="66.04" y2="55.88" width="0.1524" layer="91"/>
-<label x="66.04" y="53.34" size="1.778" layer="95"/>
+<label x="60.96" y="63.5" size="1.778" layer="95" rot="R90"/>
+<wire x1="58.42" y1="63.5" x2="58.42" y2="71.12" width="0.1524" layer="91"/>
+<pinref part="SENS" gate="G$1" pin="B"/>
 </segment>
 </net>
@@
 </segment>
 <segment>
-<pinref part="SWEEP_DIR" gate="G$1" pin="COM1"/>
-<wire x1="109.22" y1="139.7" x2="121.92" y2="139.7" width="0.1524" layer="91"/>
-<label x="119.38" y="139.7" size="1.778" layer="95"/>
+<label x="116.84" y="127" size="1.778" layer="95"/>
+<wire x1="109.22" y1="129.54" x2="121.92" y2="129.54" width="0.1524" layer="91"/>
+<pinref part="SWEEP_DIR" gate="G$1" pin="COM2"/>
 </segment>
 </net>
@@
 </segment>
 <segment>
-<pinref part="SWEEP_DIR" gate="G$1" pin="COM2"/>
-<wire x1="109.22" y1="129.54" x2="121.92" y2="129.54" width="0.1524" layer="91"/>
-<label x="119.38" y="129.54" size="1.778" layer="95"/>
+<label x="119.38" y="139.7" size="1.778" layer="95"/>
+<wire x1="109.22" y1="139.7" x2="121.92" y2="139.7" width="0.1524" layer="91"/>
+<pinref part="SWEEP_DIR" gate="G$1" pin="COM1"/>
 </segment>
 </net>

Commit message: sdsds
Connections:
- removed net N$1: 470.2, SWEEP_DIR.A1, SWEEP_DIR.B2
- new net N$2: 470.2, SWEEP_DIR.A2, SWEEP_DIR.B1
- net SWEEP_B: now also SWEEP_DIR.A1, SWEEP_DIR.B2; no longer SWEEP_DIR.A2, SWEEP_DIR.B1
Other:
- moved on the sheet: 470
Changed lines of the file:
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@@
 <instance part="GND10" gate="1" x="111.76" y="121.92"/>
 <instance part="GND11" gate="1" x="111.76" y="88.9"/>
-<instance part="470" gate="G$1" x="86.36" y="116.84" rot="R90"/>
+<instance part="470" gate="G$1" x="88.9" y="111.76" rot="R90"/>
 <instance part="JP1" gate="G$1" x="121.92" y="-27.94"/>
 <instance part="MRAT" gate="A" x="76.2" y="-68.58" smashed="yes">
@@
 <segment>
 <pinref part="470" gate="G$1" pin="1"/>
-<wire x1="86.36" y1="111.76" x2="86.36" y2="109.22" width="0.1524" layer="91"/>
+<wire x1="88.9" y1="106.68" x2="88.9" y2="101.6" width="0.1524" layer="91"/>
 <label x="83.82" y="106.68" size="1.778" layer="95"/>
 </segment>
@@
 </segment>
 </net>
-<net name="N$1" class="0">
-<segment>
-<pinref part="SWEEP_DIR" gate="G$1" pin="B2"/>
-<wire x1="93.98" y1="127" x2="86.36" y2="127" width="0.1524" layer="91"/>
-<wire x1="86.36" y1="127" x2="86.36" y2="142.24" width="0.1524" layer="91"/>
-<pinref part="SWEEP_DIR" gate="G$1" pin="A1"/>
-<wire x1="86.36" y1="142.24" x2="93.98" y2="142.24" width="0.1524" layer="91"/>
-<pinref part="470" gate="G$1" pin="2"/>
-<wire x1="86.36" y1="121.92" x2="86.36" y2="127" width="0.1524" layer="91"/>
-<junction x="86.36" y="127"/>
-</segment>
-</net>
 <net name="SWEEP_B" class="0">
 <segment>
@@
 </segment>
 <segment>
+<label x="68.58" y="137.16" size="1.778" layer="95"/>
+<junction x="83.82" y="137.16"/>
+<wire x1="86.36" y1="137.16" x2="83.82" y2="137.16" width="0.1524" layer="91"/>
+<wire x1="83.82" y1="137.16" x2="73.66" y2="137.16" width="0.1524" layer="91"/>
+<pinref part="SWEEP_DIR" gate="G$1" pin="B2"/>
+<wire x1="93.98" y1="127" x2="86.36" y2="127" width="0.1524" layer="91"/>
+<wire x1="86.36" y1="127" x2="86.36" y2="137.16" width="0.1524" layer="91"/>
+<pinref part="SWEEP_DIR" gate="G$1" pin="A1"/>
+<wire x1="86.36" y1="137.16" x2="86.36" y2="142.24" width="0.1524" layer="91"/>
+<wire x1="86.36" y1="142.24" x2="93.98" y2="142.24" width="0.1524" layer="91"/>
+<junction x="86.36" y="137.16"/>
+</segment>
+</net>
+<net name="N$2" class="0">
+<segment>
+<pinref part="470" gate="G$1" pin="2"/>
+<wire x1="88.9" y1="116.84" x2="88.9" y2="132.08" width="0.1524" layer="91"/>
+<pinref part="SWEEP_DIR" gate="G$1" pin="B1"/>
+<wire x1="88.9" y1="137.16" x2="93.98" y2="137.16" width="0.1524" layer="91"/>
 <pinref part="SWEEP_DIR" gate="G$1" pin="A2"/>
 <wire x1="93.98" y1="132.08" x2="88.9" y2="132.08" width="0.1524" layer="91"/>
 <wire x1="88.9" y1="132.08" x2="88.9" y2="137.16" width="0.1524" layer="91"/>
-<pinref part="SWEEP_DIR" gate="G$1" pin="B1"/>
-<wire x1="88.9" y1="137.16" x2="93.98" y2="137.16" width="0.1524" layer="91"/>
-<wire x1="88.9" y1="137.16" x2="81.28" y2="137.16" width="0.1524" layer="91"/>
-<junction x="88.9" y="137.16"/>
-<label x="68.58" y="137.16" size="1.778" layer="95"/>
-</segment>
-</net>
+<junction x="88.9" y="132.08"/>
+</segment>
+</net>
