File: panel/pclone2_panel.sch (EAGLE design)
At the start: 22 parts

Commit message: v2 - smt headers
Parts:
- removed ADECAY, CLK, MDEP, MRAT, TSENS, VPITCH, VSHP: (no value), pinhead:PINHD-1X3
- removed MSHP, TIN: (no value), pinhead:PINHD-1X2
- removed VSWP: (no value), pinhead:PINHD-1X4
- added JP2: (no value), microbuilder:HEADER-1X5SMT
- added JP3, JP4: (no value), microbuilder:HEADER-1X10SMT
- added JP5: (no value), microbuilder:HEADER-1X3SMT
- added JP6: (no value), jason_eagle6:PINHD-1X1SMT
Connections:
- net CLICK1: now also JP2.1; no longer CLK.2
- net CLICK2: now also JP2.2; no longer CLK.3
- net DECAY: now also JP3.7, JP3.8; no longer ADECAY.2, ADECAY.3
- net DEPTH1: now also JP4.6; no longer MDEP.1
- net DEPTH2: now also JP4.7; no longer MDEP.2
- net DEPTH3: now also JP4.8; no longer MDEP.3
- net GND: now also JP3.1, JP3.3, JP3.6, JP6.1; no longer ADECAY.1, CLK.1, TIN.1, TSENS.1
- net MODRATE1: now also JP5.1; no longer MRAT.1
- net MODRATE2: now also JP5.2; no longer MRAT.2
- net MODRATE3: now also JP5.3; no longer MRAT.3
- net MODSHAPE1: now also JP4.9; no longer MSHP.1
- net MODSHAPE2: now also JP4.10; no longer MSHP.2
- net PITCH1: now also JP3.9; no longer VPITCH.1
- net PITCH2: now also JP3.10; no longer VPITCH.2
- net PITCH3: now also JP4.1; no longer VPITCH.3
- net SENS2: now also JP3.4; no longer TSENS.2
- net SENS3: now also JP3.5; no longer TSENS.3
- net SWEEP1: now also JP4.2; no longer VSWP.1
- net SWEEP2: now also JP4.3; no longer VSWP.2
- net SWEEP3: now also JP4.4; no longer VSWP.3
- net SWEEP4: now also JP4.5; no longer VSWP.4
- net TRIG2: now also JP3.2; no longer TIN.2
- net VCOWAVE1: now also JP2.3; no longer VSHP.1
- net VCOWAVE2: now also JP2.4; no longer VSHP.2
- net VCOWAVE3: now also JP2.5; no longer VSHP.3
Other:
- moved on the sheet: JP1
